File: kicad/pdice-04/pdice-04.kicad_sch (KiCad schematic)
At the start: 29 parts, among them J1 Conn_01x06, J2 USB_C_Receptacle_PowerOnly_6P, J3 Conn_01x02, SW1 SW_Slide, SW2 SW_Push, SW3 SW_Slide, U1 PIC12F1572, U2 74HC164

Commit message: Created construction manual and updated schematics with part numbers
Parts:
- C1: OC_MOUSER (none) -> 81-GCM188R71H104KA7D
- LOGO1: now left out of the parts list
- R1, R2: OC_MOUSER (none) -> 594-MCT06030C5101FP5
- R3: OC_MOUSER (none) -> 594-MCT06030C4702FP5
- R4: OC_MOUSER (none) -> 594-MCT06030Z0000ZP5
- SW1, SW3: OC_MOUSER (none) -> 612-EG1218
Other:
- note added: "Dobbelsteen Alle LEDs 2mA type (Low Current) Rood: WP7113LID Geel: LTL2R3KYD-EM Groen: LTL2R3KGD-EM"
- note removed: "Dobbelsteen Alle LEDs 2mA type (Low Current), Rood: WP7113LID Geel: LTL2R3KYD-EM Groen: LTL2R3KGD-EM"
Changed lines of the file:
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@@
 		(title "Dobbelsteen met PIC12 microcontroller")
 		(date "2026-09-12")
-		(rev "0.1")
+		(rev "0.4")
 		(company "Elektronica Beta VU")
 		(comment 1 "Vrije Universiteit Amsterdam")
@@
 		)
 	)
-	(text "Dobbelsteen\nAlle LEDs 2mA type (Low Current),\nRood: WP7113LID\nGeel: LTL2R3KYD-EM\nGroen: LTL2R3KGD-EM "
+	(text "Dobbelsteen\nAlle LEDs 2mA type (Low Current)\nRood: WP7113LID\nGeel: LTL2R3KYD-EM\nGroen: LTL2R3KGD-EM "
 		(exclude_from_sim no)
 		(at 245.745 142.875 0)
@@
 		(body_style 1)
 		(exclude_from_sim no)
-		(in_bom yes)
+		(in_bom no)
 		(on_board yes)
 		(in_pos_files yes)
@@
 			)
 		)
+		(property "MFG" ""
+			(at 154.94 180.34 0)
+			(hide yes)
+			(show_name no)
+			(do_not_autoplace no)
+			(effects
+				(font
+					(size 1.27 1.27)
+				)
+			)
+		)
+		(property "MPN" ""
+			(at 154.94 180.34 0)
+			(hide yes)
+			(show_name no)
+			(do_not_autoplace no)
+			(effects
+				(font
+					(size 1.27 1.27)
+				)
+			)
+		)
+		(property "OC_MOUSER" ""
+			(at 154.94 180.34 0)
+			(hide yes)
+			(show_name no)
+			(do_not_autoplace no)
+			(effects
+				(font
+					(size 1.27 1.27)
+				)
+			)
+		)
+		(property "OC_RS" ""
+			(at 154.94 180.34 0)
+			(hide yes)
+			(show_name no)
+			(do_not_autoplace no)
+			(effects
+				(font
+					(size 1.27 1.27)
+				)
+			)
+		)
+		(property "OC_FARNELL" ""
+			(at 154.94 180.34 0)
+			(hide yes)
+			(show_name no)
+			(do_not_autoplace no)
+			(effects
+				(font
+					(size 1.27 1.27)
+				)
+			)
+		)
+		(property "OC_CONRAD" ""
+			(at 154.94 180.34 0)
+			(hide yes)
+			(show_name no)
+			(do_not_autoplace no)
+			(effects
+				(font
+					(size 1.27 1.27)
+				)
+			)
+		)
 		(instances
 			(project "pdice-04"
@@
 			)
 		)
+		(property "OC_MOUSER" "594-MCT06030Z0000ZP5"
+			(at 138.43 116.84 90)
+			(hide yes)
+			(show_name no)
+			(do_not_autoplace no)
+			(effects
+				(font
+					(size 1.27 1.27)
+				)
+			)
+		)
 		(pin "2"
 		)
@@
 			)
 		)
+		(property "OC_MOUSER" "594-MCT06030C4702FP5"
+			(at 72.39 105.41 0)
+			(hide yes)
+			(show_name no)
+			(do_not_autoplace no)
+			(effects
+				(font
+					(size 1.27 1.27)
+				)
+			)
+		)
 		(pin "2"
 		)
@@
 			)
 		)
+		(property "OC_MOUSER" "81-GCM188R71H104KA7D"
+			(at 87.63 138.43 0)
+			(hide yes)
+			(show_name no)
+			(do_not_autoplace no)
+			(effects
+				(font
+					(size 1.27 1.27)
+				)
+			)
+		)
 		(pin "1"
 		)
@@
 			(at 33.655 55.88 90)
 			(show_name no)
-			(do_not_autoplace no)
+			(do_not_autoplace yes)
 			(effects
 				(font
@@
 			)
 		)
-		(property "OC_MOUSER" ""
+		(property "OC_MOUSER" "612-EG1218"
 			(at 74.93 45.72 0)
 			(hide yes)
@@
 			)
 		)
-		(property "OC_MOUSER" ""
+		(property "OC_MOUSER" "594-MCT06030C5101FP5 "
 			(at 63.5 68.58 0)
 			(hide yes)
@@
 			)
 		)
+		(property "OC_MOUSER" "594-MCT06030C5101FP5 "
+			(at 69.85 68.58 0)
+			(hide yes)
+			(show_name no)
+			(do_not_autoplace no)
+			(effects
+				(font
+					(size 1.27 1.27)
+				)
+			)
+		)
 		(pin "2"
 		)
@@
 			)
 		)
-		(property "OC_MOUSER" ""
+		(property "OC_MOUSER" "612-EG1218"
 			(at 151.13 139.7 0)
 			(hide yes)
